Commit message: feat: update to humble & add docker
Signed-off-by: Amadeusz Szymko <amadeuszszymko@gmail.com>

File: phoxi_camera_ros2/urdf/M+_Motion_Cam-3D.xacro (robot description, xacro)
@@ -2,5 +2,5 @@
 <robot name="phoxi" xmlns:xacro="http://ros.org/wiki/xacro">
   <xacro:arg name="config_dir" default="$(find phoxi_camera_ros2)/param"/>
-  <xacro:property name="config" value="${load_yaml('$(arg config_dir)/defaults.param.yaml')}"/>
+  <xacro:property name="config" value="${xacro.load_yaml('$(arg config_dir)/defaults.param.yaml')}"/>
   <xacro:include filename="phoxi.xacro"/>
   <xacro:phoxi_macro
